File: KiCad/Agnus_8375/Agnus.kicad_pcb (KiCad board)
At the start: 4 copper layers, 28.9 x 28.9 mm, 35 parts, among them J6 Conn_01x01, U1 10M02SCU169C8G, U2 LM1117-3.3, U3 SN74CBTD16210, U4 SN74CBTD16210, U5 SN74CBTD16210, U6 SN74CBTD16210, U7 Agnus_8375_MB_socket

Commit message: changed D2,E2 from NC to GND, D3 from NC to 3V3
Connections:
- U1 pad D2: Net-(U1-PadD2) -> GND
- U1 pad D3: Net-(U1-PadD3) -> 3V3
- U1 pad E2: Net-(U1-PadE2) -> GND
Routing:
- net GND: track 231.1 -> 233.6 mm
- net 3V3: track 154.6 -> 155.9 mm
