File: KiCad/Agnus_8375/Agnus_FPGA.sch (KiCad schematic (older format))
At the start: 26 parts, among them J6 Conn_01x01, U1 10M02SCU169C8G, U2 LM1117-3.3

Commit message: changed D2,E2 from NC to GND, D3 from NC to 3V3
Connections:
- net 3V3: now also U1.K4 (VCCA1)
- net GND: now also U1.D2 (GND), U1.E2 (GND)
Changed lines of the file:
@@
 U 1 1 60A0E571
 P 3400 3700
+AR Path="/60A0E571" Ref="U1"  Part="1"
+AR Path="/608A10F5/60A0E571" Ref="U1"  Part="1"
 F 0 "U1" H 3400 3750 60  0000 C CNN
 F 1 "10M02SCU169C8G" H 3400 3900 60  0000 C CNN
@@
 	2800 1250 2900 1250
 Wire Wire Line
-	3500 800  3500 1250
-Wire Wire Line
-	2900 800  3500 800
+	3400 800  3400 1250
+Wire Wire Line
+	2900 800  3400 800
 Wire Wire Line
 	3500 1250 3600 1250
-Connection ~ 3500 1250
 Connection ~ 3600 1250
 Wire Wire Line
@@
 Wire Wire Line
 	8100 1500 8500 1500
+Wire Wire Line
+	3400 1250 3500 1250
+Connection ~ 3400 1250
+Connection ~ 3500 1250
+Wire Wire Line
+	4100 4550 4200 4550
+Connection ~ 4100 4550
+Connection ~ 4200 4550
+Wire Wire Line
+	4200 4550 4300 4550
 $EndSCHEMATC
